Commit message: Fixes coordintate frame issues in ardupilot code and URDF.

File: igvc/launch/test_platform.urdf (robot description, URDF)
Before this commit: robot test_platform, 6 links, 5 joints
Joints:
- joint imu: origin xyz=0 -0.11 1.083 rpy=0 0 0 -> xyz=0 -0.11 1.083 rpy=0 0 -1.570796326

Commit message: Position tracker work.

File: igvc/launch/test_platform.urdf (robot description, URDF)
Before this commit: robot test_platform, 6 links, 5 joints
Joints:
- joint imu: origin xyz=0 -0.11 1.083 rpy=0 0 -1.570796326 -> xyz=0 -0.11 1.083 rpy=0 0 0

Commit message: Added mapper needs to be tested more and optimized

File: igvc/launch/test_platform.urdf (robot description, URDF)
Before this commit: robot test_platform, 6 links, 5 joints
Links:
- added link camera_left
- added link camera_right
Joints:
- added joint camera_left: type fixed, parent camera, child camera_left, origin xyz=-0.051 0 0 rpy=0 0 0, axis 0 0 0
- added joint camera_right: type fixed, parent camera, child camera_right, origin xyz=0.051 0 0 rpy=0 0 0, axis 0 0 0

Commit message: Rotates lidar 90 degrees in tf and removes some comments in map main.cpp

File: igvc/launch/test_platform.urdf (robot description, URDF)
Before this commit: robot test_platform, 8 links, 7 joints
Joints:
- joint lidar: origin xyz=0 0.52 0.243 rpy=0 0 0 -> xyz=0 0.52 0.243 rpy=0 0 1.5707
