Commit message: Changed method to project camera points using TF system, corrected camera pose

File: igvc/launch/mistii.urdf (robot description, URDF)
Before this commit: robot test_platform, 8 links, 7 joints
Joints:
- joint camera: origin xyz=0 -0.18 1.34 rpy=-0.3491 0 0 -> xyz=0 -0.18 1.34 rpy=-1.9199 0 0

Commit message: Localized 3 cameras

File: igvc/launch/mistii.urdf (robot description, URDF)
Before this commit: robot test_platform, 8 links, 7 joints
Links:
- removed link camera
- removed link camera_left
- removed link camera_right
- added link usb_cam_center
- added link usb_cam_left
- added link usb_cam_right
Joints:
- removed joint camera
- removed joint camera_left
- removed joint camera_right
- added joint usb_cam_center: type fixed, parent base_link, child usb_cam_center, origin xyz=-0.0549131 -.117477 1.50282 rpy=-1.89853 -.0193608 0.0194719, axis 0 0 0
- added joint usb_cam_left: type fixed, parent base_footprint, child usb_cam_left, origin xyz=-0.115369 -0.0331363 1.82578 rpy=-2.89953 -.814402 1.69177, axis 0 0 0
- added joint usb_cam_right: type fixed, parent base_footprint, child usb_cam_right, origin xyz=.348438 -0.190612 1.3478 rpy=-2.85843 0.900295 -1.58223, axis 0 0 0
- joint lidar: origin xyz=0 0.83 0.455 rpy=0 0 1.5707 -> xyz=0 0.83 0.0 rpy=0 0 1.5707; parent base_link -> base_footprint
