Commit message: added plugin for the lidar and added necessary nodes to the gazebo launch file for the robot state publisher'

File: gazebo/igvc_description/urdf/Jaymii.urdf (robot description, URDF)
Before this commit: robot Jaymii, 13 links, 12 joints
Links:
- removed link lidar_link
- added link base_footprint
- added link lidar; visual cylinder length=0.1 radius=0.05
Joints:
- added joint groundToDriveWheelMidpoint: type fixed, parent base_footprint, child base_link, origin xyz=0 0 0.17 rpy=0 0 0, axis 0 0 0
- joint body_to_lidar: child lidar_link -> lidar

Commit message: fixed camera topic to be center not main and added plugin for movement

File: gazebo/igvc_description/urdf/Jaymii.urdf (robot description, URDF)
Before this commit: robot Jaymii, 14 links, 13 joints
Links:
- removed link main_camera_link
- added link center_camera_link; visual box size=0.1 0.1 0.1
Joints:
- removed joint body_to_main_camera
- added joint body_to_center_camera: type fixed, parent body, child center_camera_link, origin xyz=0.15 0 1.2 rpy=0 0 0

Commit message: added transmission and removed visualize from gazebo

File: gazebo/igvc_description/urdf/Jaymii.urdf (robot description, URDF)
Before this commit: robot Jaymii, 14 links, 13 joints
Joints:
- removed joint bady_to_back_ball
- added joint body_to_back_ball: type floating, parent body, child back_ball, origin xyz=-0.381 0 -0.0125 rpy=0 0 0

Commit message: Changed urdf camera link names for lookuptransform

File: gazebo/igvc_description/urdf/Jaymii.urdf (robot description, URDF)
Before this commit: robot Jaymii, 14 links, 13 joints
Links:
- removed link center_camera_link
- removed link left_camera_link
- removed link right_camera_link
- added link usb_cam_center; visual box size=0.1 0.1 0.1
- added link usb_cam_left; visual box size=0.1 0.1 0.1
- added link usb_cam_right; visual box size=0.1 0.1 0.1
Joints:
- joint body_to_center_camera: child center_camera_link -> usb_cam_center
- joint body_to_left_camera: child left_camera_link -> usb_cam_left
- joint body_to_right_camera: child right_camera_link -> usb_cam_right

Commit message: changed frame names and topic names to match bag file

File: gazebo/igvc_description/urdf/Jaymii.urdf (robot description, URDF)
Before this commit: robot Jaymii, 14 links, 13 joints
Joints:
- joint body_to_imu: origin xyz=0.25 0 0.5 rpy=0 0 0 -> xyz=0.0 1.3462 0.0  rpy=0 0 0; parent body -> axle

Commit message: rotated imu to match rest of URDF

File: gazebo/igvc_description/urdf/Jaymii.urdf (robot description, URDF)
Before this commit: robot Jaymii, 14 links, 13 joints
Joints:
- joint body_to_imu: origin xyz=0.0 1.3462 0.0  rpy=0 0 0 -> xyz=0.0 1.3462 0.0  rpy=-1.5708 0 0

Commit message: added _optical links to camera to account for transform

File: gazebo/igvc_description/urdf/Jaymii.urdf (robot description, URDF)
Before this commit: robot Jaymii, 14 links, 13 joints
Links:
- added link center_camera_optical
- added link left_camera_optical
- added link right_camera_optical
Joints:
- added joint camera_center_optical_joint: type fixed, parent center_camera_link, child center_camera_optical, origin xyz=0 0 0 rpy=-1.5708 0 -1.5708
- added joint camera_left_optical_joint: type fixed, parent left_camera_link, child left_camera_optical, origin xyz=0 0 0 rpy=-1.5708 0 -1.5708
- added joint camera_right_optical_joint: type fixed, parent right_camera_link, child right_camera_optical, origin xyz=0 0 0 rpy=-1.5708 0 -1.5708

Commit message: fixed issues

File: gazebo/igvc_description/urdf/Jaymii.urdf (robot description, URDF)
Before this commit: robot Jaymii, 17 links, 16 joints
Links:
- removed link usb_cam_center
- removed link usb_cam_left
- removed link usb_cam_right
- added link center_camera_link; visual box size=0.1 0.1 0.1
- added link left_camera_link; visual box size=0.1 0.1 0.1
- added link right_camera_link; visual box size=0.1 0.1 0.1
Joints:
- joint body_to_center_camera: child usb_cam_center -> center_camera_link
- joint body_to_left_camera: child usb_cam_left -> left_camera_link
- joint body_to_right_camera: child usb_cam_right -> right_camera_link

Commit message: improvements to Gazebo, fixed gps data, still need to fix imu

File: gazebo/igvc_description/urdf/Jaymii.urdf (robot description, URDF)
Before this commit: robot Jaymii, 17 links, 16 joints
Links:
- removed link gps_link
- removed link imu_link
- added link gps; visual cylinder length=0.05 radius=0.1
- added link imu; visual box size=0.1 0.1 0.1
Joints:
- joint axle_to_left_wheel: origin xyz=0 0 0.3175 rpy=0 0 0 -> xyz=0 0 -0.3175 rpy=0 0 0
- joint axle_to_right_wheel: origin xyz=0 0 -0.3175 rpy=0 0 0 -> xyz=0 0 0.3175 rpy=0 0 0
- joint body_to_gps: child gps_link -> gps
- joint body_to_imu: child imu_link -> imu; origin xyz=0.0 1.3462 0.0  rpy=-1.5708 0 0 -> xyz=0 0 1.3 rpy=0 0 -1.5708; parent axle -> body
- joint groundToDriveWheelMidpoint: origin xyz=0 0 0.17 rpy=0 0 0 -> xyz=0 0 0 rpy=0 0 0

Commit message: rotated imu so everything is consistent, pathplanner still has x and y flipped when it generates the resulting location

File: gazebo/igvc_description/urdf/Jaymii.urdf (robot description, URDF)
Before this commit: robot Jaymii, 17 links, 16 joints
Joints:
- joint base_link_to_body: axis 0 -1 -1 -> (none)
- joint body_to_imu: origin xyz=0 0 1.3 rpy=0 0 -1.5708 -> xyz=0 0 1.3 rpy=0 0 0

Commit message: removed URDF namesapce from topic names

File: gazebo/igvc_description/urdf/Jaymii.urdf (robot description, URDF)
Before this commit: robot Jaymii, 17 links, 16 joints
Links:
- removed link center_camera_link
- removed link left_camera_link
- removed link right_camera_link
- added link usb_cam_center; visual box size=0.1 0.1 0.1
- added link usb_cam_left; visual box size=0.1 0.1 0.1
- added link usb_cam_right; visual box size=0.1 0.1 0.1
Joints:
- removed joint camera_center_optical_joint
- removed joint camera_left_optical_joint
- removed joint camera_right_optical_joint
- added joint optical_cam_center: type fixed, parent usb_cam_center, child center_camera_optical, origin xyz=0 0 0 rpy=-1.5708 0 -1.5708
- added joint optical_cam_left: type fixed, parent usb_cam_left, child left_camera_optical, origin xyz=0 0 0 rpy=-1.5708 0 -1.5708
- added joint optical_cam_right: type fixed, parent usb_cam_right, child right_camera_optical, origin xyz=0 0 0 rpy=-1.5708 0 -1.5708
- joint body_to_center_camera: child center_camera_link -> usb_cam_center
- joint body_to_left_camera: child left_camera_link -> usb_cam_left
- joint body_to_right_camera: child right_camera_link -> usb_cam_right

Commit message: fixed camera link names for optical

File: gazebo/igvc_description/urdf/Jaymii.urdf (robot description, URDF)
Before this commit: robot Jaymii, 17 links, 16 joints
Links:
- removed link center_camera_optical
- removed link left_camera_optical
- removed link right_camera_optical
- added link optical_cam_center
- added link optical_cam_left
- added link optical_cam_right
Joints:
- removed joint optical_cam_center
- removed joint optical_cam_left
- removed joint optical_cam_right
- added joint optical_cam_center_joint: type fixed, parent usb_cam_center, child optical_cam_center, origin xyz=0 0 0 rpy=-1.5708 0 -1.5708
- added joint optical_cam_left_joint: type fixed, parent usb_cam_left, child optical_cam_left, origin xyz=0 0 0 rpy=-1.5708 0 -1.5708
- added joint optical_cam_right_joint: type fixed, parent usb_cam_right, child optical_cam_right, origin xyz=0 0 0 rpy=-1.5708 0 -1.5708

Commit message: implemented a lcoal occupancy grid centered at the robot, tuned donw the pid, made base footprint the base of the robot instead of the center

File: gazebo/igvc_description/urdf/Jaymii.urdf (robot description, URDF)
Before this commit: robot Jaymii, 17 links, 16 joints
Joints:
- joint groundToDriveWheelMidpoint: origin xyz=0 0 0 rpy=0 0 0 -> xyz=0 0 0.12 rpy=0 0 0

Commit message: fixed gps and center camera location, altered the wheels and balls based off of the CAD model due to inconsistencies this may need to be changed

File: gazebo/igvc_description/urdf/Jaymii.urdf (robot description, URDF)
Before this commit: robot Jaymii, 17 links, 16 joints
Joints:
- joint axle_to_left_wheel: origin xyz=0 0 -0.3175 rpy=0 0 0 -> xyz=0 0 -0.3177286 rpy=0 0 0
- joint axle_to_right_wheel: origin xyz=0 0 0.3175 rpy=0 0 0 -> xyz=0 0 0.3177286 rpy=0 0 0
- joint body_to_back_ball: origin xyz=-0.381 0 -0.0125 rpy=0 0 0 -> xyz=-0.385064 0 -0.0125 rpy=0 0 0
- joint body_to_center_camera: origin xyz=0.15 0 1.2 rpy=0 0 0 -> xyz=0.05 0 1.3843 rpy=0 0 0
- joint body_to_front_ball: origin xyz=0.381 0 -0.0125 rpy=0 0 0 -> xyz=0.385064 0 -0.0125 rpy=0 0 0
- joint body_to_gps: origin xyz=0.25 0.1 0.5 rpy=0 0 0 -> xyz=0 0.1166876 0.5225542 rpy=0 0 0

Commit message: fixed lidar location according to the CAD

File: gazebo/igvc_description/urdf/Jaymii.urdf (robot description, URDF)
Before this commit: robot Jaymii, 17 links, 16 joints
Joints:
- joint body_to_lidar: origin xyz=0.45 0 0.5 rpy=0 0 0 -> xyz=0.45 0 0.6435344 rpy=0 0 0

Commit message: updated the URDF to match teh CAD model, all sensors should be in the correct palce now

File: gazebo/igvc_description/urdf/Jaymii.urdf (robot description, URDF)
Before this commit: robot Jaymii, 17 links, 16 joints
Joints:
- removed joint base_link_to_body
- removed joint body_to_axle
- removed joint body_to_back_ball
- removed joint body_to_center_camera
- removed joint body_to_front_ball
- removed joint body_to_gps
- removed joint body_to_imu
- removed joint body_to_lidar
- removed joint groundToDriveWheelMidpoint
- added joint base_footprint_to_axle: type fixed, parent base_footprint, child axle, origin xyz=0 0 0.1651 rpy=1.5708 0 0
- added joint base_footprint_to_back_ball: type floating, parent base_footprint, child back_ball, origin xyz=-0.385064 0 0.1016 rpy=0 0 0
- added joint base_footprint_to_base_link: type fixed, parent base_footprint, child base_link, origin xyz=0 0 0.12 rpy=0 0 0, axis 0 0 0
- added joint base_footprint_to_body: type fixed, parent base_footprint, child body, origin xyz=0 0 0.12 rpy=0 0 0
- added joint base_footprint_to_center_camera: type fixed, parent base_footprint, child usb_cam_center, origin xyz=0.03302 0 1.5875 rpy=0 0 0
- added joint base_footprint_to_front_ball: type floating, parent base_footprint, child front_ball, origin xyz=0.385064 0 0.1016 rpy=0 0 0
- added joint base_footprint_to_gps: type fixed, parent base_footprint, child gps, origin xyz=-0.04572 0.2032 0.7112 rpy=0 0 0
- added joint base_footprint_to_imu: type fixed, parent base_footprint, child imu, origin xyz=0.12192 0 0.64516 rpy=0 0 0
- added joint base_footprint_to_lidar: type fixed, parent base_footprint, child lidar, origin xyz=0.50038 0 0.69596 rpy=0 0 0
- joint axle_to_left_wheel: origin xyz=0 0 -0.3177286 rpy=0 0 0 -> xyz=0 0 -0.32004 rpy=0 0 0
- joint axle_to_right_wheel: origin xyz=0 0 0.3177286 rpy=0 0 0 -> xyz=0 0 0.32004 rpy=0 0 0

Commit message: updated URDF to account for the new robot

File: gazebo/igvc_description/urdf/Jaymii.urdf (robot description, URDF)
Before this commit: robot Jaymii, 17 links, 16 joints
Joints:
- joint base_footprint_to_center_camera: origin xyz=0.03302 0 1.5875 rpy=0 0 0 -> xyz=0.03302 0 1.7145 rpy=0 0 0
- joint base_footprint_to_gps: origin xyz=-0.04572 0.2032 0.7112 rpy=0 0 0 -> xyz=-0.04572 0.2032 0.9525 rpy=0 0 0
- joint base_footprint_to_imu: origin xyz=0.12192 0 0.64516 rpy=0 0 0 -> xyz=0.12192 0 0.9525 rpy=0 0 0
- joint base_footprint_to_lidar: origin xyz=0.50038 0 0.69596 rpy=0 0 0 -> xyz=0.4572 0 0.9525 rpy=0 0 0

Commit message: imu is centrally located now

File: gazebo/igvc_description/urdf/Jaymii.urdf (robot description, URDF)
Before this commit: robot Jaymii, 17 links, 16 joints
Joints:
- joint base_footprint_to_imu: origin xyz=0.12192 0 0.9525 rpy=0 0 0 -> xyz=0.0 0 0.9525 rpy=0 0 0

Commit message: rotated imu in URDF to get correct orientation for the real robot

File: gazebo/igvc_description/urdf/Jaymii.urdf (robot description, URDF)
Before this commit: robot Jaymii, 17 links, 16 joints
Joints:
- joint base_footprint_to_imu: origin xyz=0.0 0 0.9525 rpy=0 0 0 -> xyz=0.0 0 0.9525 rpy=0 0 3.141

Commit message: created new tf tree

File: gazebo/igvc_description/urdf/Jaymii.urdf (robot description, URDF)
Before this commit: robot Jaymii, 17 links, 16 joints
Joints:
- removed joint axle_to_left_wheel
- removed joint axle_to_right_wheel
- removed joint base_footprint_to_axle
- removed joint base_footprint_to_base_link
- removed joint base_footprint_to_body
- removed joint base_footprint_to_center_camera
- removed joint base_footprint_to_gps
- removed joint base_footprint_to_imu
- removed joint base_footprint_to_lidar
- removed joint body_to_left_camera
- removed joint body_to_right_camera
- added joint imu_to_base_footprint: type fixed, parent imu, child base_footprint, origin xyz=0 0 -.633 rpy=0 0 0, axis 0 0 0
- added joint imu_to_center_camera: type fixed, parent imu, child usb_cam_center, origin xyz=-.056 0 .937 rpy=0 0 0
- added joint imu_to_gps: type fixed, parent imu, child gps, origin xyz=-.044 .214 0 rpy=0 0 0
- added joint imu_to_left_wheel: type fixed, parent imu, child left_wheel, origin xyz=-.287 .444 -.465 rpy=0 0 3.141
- added joint imu_to_lidar: type fixed, parent imu, child lidar, origin xyz=.276 -.029 .029 rpy=0 0 0
- added joint imu_to_right_wheel: type fixed, parent imu, child right_wheel, origin xyz=-.287 -.438 -.465 rpy=0 0 0

Commit message: New TF tree

File: gazebo/igvc_description/urdf/Jaymii.urdf (robot description, URDF)
Before this commit: robot Jaymii, 17 links, 11 joints
Joints:
- joint imu_to_center_camera: origin xyz=-.056 0 .937 rpy=0 0 0 -> xyz=-.056 0 .937 rpy=0 1.03 0

Commit message: Fixed TF tree and renamed node

File: gazebo/igvc_description/urdf/Jaymii.urdf (robot description, URDF)
Before this commit: robot Jaymii, 17 links, 11 joints
Links:
- removed link base_link
- removed link body
- removed link optical_cam_left
- removed link optical_cam_right
- removed link usb_cam_left
- removed link usb_cam_right
Joints:
- removed joint base_footprint_to_back_ball
- removed joint base_footprint_to_front_ball
- removed joint imu_to_left_wheel
- removed joint imu_to_right_wheel
- removed joint optical_cam_left_joint
- removed joint optical_cam_right_joint
- added joint axle_to_left_wheel: type fixed, parent axle, child left_wheel, origin xyz=0 0 .222 rpy=0 0 3.141
- added joint axle_to_right_wheel: type fixed, parent axle, child right_wheel, origin xyz=0 0 -.219 rpy=0 0 0
- added joint imu_to_axle: type fixed, parent imu, child axle, origin xyz=-.287 -.003 -.465 rpy=1.5708 0 0, axis 0 0 0
- added joint imu_to_back_ball: type floating, parent imu, child back_ball, origin xyz=-0.385064 0 0.1016 rpy=0 0 0
- added joint imu_to_front_ball: type floating, parent imu, child front_ball, origin xyz=0.385064 0 0.1016 rpy=0 0 0

Commit message: Adjusted tf-tree

File: gazebo/igvc_description/urdf/Jaymii.urdf (robot description, URDF)
Before this commit: robot Jaymii, 11 links, 10 joints
Links:
- added link base_link; visual box size=0.01 0.01 0.01
Joints:
- added joint base_link_to_imu: type fixed, parent base_link, child imu, origin xyz=0 0 0 rpy=0 0 0, axis 0 0 0
- joint axle_to_left_wheel: origin xyz=0 0 .222 rpy=0 0 3.141 -> xyz=0 0 -.39 rpy=0 0 3.141
- joint axle_to_right_wheel: origin xyz=0 0 -.219 rpy=0 0 0 -> xyz=0 0 .39 rpy=0 0 0
- joint imu_to_back_ball: origin xyz=-0.385064 0 0.1016 rpy=0 0 0 -> xyz=-.39 0 -.53 rpy=0 0 0
- joint imu_to_front_ball: origin xyz=0.385064 0 0.1016 rpy=0 0 0 -> xyz=.39 0 -.53 rpy=0 0 0

Commit message: New tf tree

File: gazebo/igvc_description/urdf/Jaymii.urdf (robot description, URDF)
Before this commit: robot Jaymii, 12 links, 11 joints
Joints:
- removed joint base_link_to_imu
- removed joint imu_to_base_footprint
- added joint base_footprint_to_base_link: type fixed, parent base_footprint, child base_link, origin xyz=0 0 0 rpy=0 0 0, axis 0 0 0
- added joint base_footprint_to_imu: type fixed, parent base_footprint, child imu, origin xyz=0 0 -.633 rpy=0 0 0, axis 0 0 0
- joint axle_to_left_wheel: axis (none) -> 0 0 -1; origin xyz=0 0 -.39 rpy=0 0 3.141 -> xyz=0 0 -.39 rpy=0 0 0; type fixed -> continuous
- joint axle_to_right_wheel: axis (none) -> 0 0 -1; type fixed -> continuous

Commit message: Adjusted pitch of camera; fixed base_footprint_to_imu joint to not place the base footpint half a meter underground

File: gazebo/igvc_description/urdf/Jaymii.urdf (robot description, URDF)
Before this commit: robot Jaymii, 12 links, 11 joints
Joints:
- joint base_footprint_to_imu: origin xyz=0 0 -.633 rpy=0 0 0 -> xyz=0 0 .633 rpy=0 0 0
- joint imu_to_back_ball: origin xyz=-.39 0 -.53 rpy=0 0 0 -> xyz=-.85 0 -.53 rpy=0 0 0
- joint imu_to_center_camera: origin xyz=-.056 0 .937 rpy=0 1.03 0 -> xyz=-.056 0 .937 rpy=0 .8 0

Commit message: updated urdf, moved axel down 0.01 m

File: gazebo/igvc_description/urdf/Jaymii.urdf (robot description, URDF)
Before this commit: robot Jaymii, 12 links, 11 joints
Joints:
- joint imu_to_axle: origin xyz=-.287 -.003 -.465 rpy=1.5708 0 0 -> xyz=-.287 -0.003 -.475 rpy=1.5708 0 0
