Commit message: updated urdf to be jessi not jaymii/woodi

File: gazebo/igvc_description/urdf/jessi.urdf (robot description, URDF)
Before this commit: robot Jaymii, 12 links, 11 joints
Joints:
- removed joint imu_to_center_camera
- removed joint imu_to_gps
- removed joint imu_to_lidar
- added joint base_footprint_to_center_camera: type fixed, parent base_footprint, child usb_cam_center, origin xyz=-.102 0 1.499 rpy=0 .8 0
- added joint base_footprint_to_gps: type fixed, parent base_footprint, child gps, origin xyz=-.102 .178 1.499 rpy=0 0 0
- added joint base_footprint_to_lidar: type fixed, parent base_footprint, child lidar, origin xyz=.610 -.013 .597 rpy=0 0 0
- joint base_footprint_to_imu: origin xyz=0 0 .633 rpy=0 0 0 -> xyz=-1.02 0.165 1.499 rpy=0 0 0
- joint imu_to_front_ball: origin xyz=.39 0 -.53 rpy=0 0 0 -> xyz=.39 -0 -.53 rpy=0 0 0

Commit message: fixed formatting in urdf

File: gazebo/igvc_description/urdf/jessi.urdf (robot description, URDF)
Before this commit: robot Jaymii, 12 links, 11 joints
Joints:
- joint imu_to_back_ball: origin xyz=-.85 0 -.53 rpy=0 0 0 -> xyz=-.85 0.0 -.53 rpy=0 0 0
- joint imu_to_front_ball: origin xyz=.39 -0 -.53 rpy=0 0 0 -> xyz=.39 0.0 -.53 rpy=0 0 0

Commit message: fixed IMU position for new placement

File: gazebo/igvc_description/urdf/jessi.urdf (robot description, URDF)
Before this commit: robot Jaymii, 12 links, 11 joints
Joints:
- joint base_footprint_to_imu: origin xyz=-1.02 0.165 1.499 rpy=0 0 0 -> xyz=-0.102 0.155 1.499 rpy=0 0 0

Commit message: firmware, updated gazebo files to match jessi and work well ish

File: gazebo/igvc_description/urdf/jessi.urdf (robot description, URDF)
Before this commit: robot Jaymii, 12 links, 11 joints
Links:
- removed link back_ball
- link front_ball: mass 1.0 -> 30.0; geometry collision sphere radius=0.16; visual sphere radius=0.16
- link left_wheel: mass 1.0 -> 30.0
- link right_wheel: mass 1.0 -> 30.0
Joints:
- removed joint imu_to_axle
- removed joint imu_to_back_ball
- removed joint imu_to_front_ball
- added joint base_footprint_to_axle: type fixed, parent base_footprint, child axle, origin xyz=0 0 0.18 rpy=1.5708 0 0, axis 0 0 0
- added joint base_footprint_to_front_ball: type floating, parent base_footprint, child front_ball, origin xyz=.610 0.0 0.18 rpy=0 0 0
- joint axle_to_left_wheel: origin xyz=0 0 -.39 rpy=0 0 0 -> xyz=0 0 -.26 rpy=0 0 0
- joint axle_to_right_wheel: origin xyz=0 0 .39 rpy=0 0 0 -> xyz=0 0 .26 rpy=0 0 0

Commit message: updated urdf

File: gazebo/igvc_description/urdf/jessi.urdf (robot description, URDF)
Before this commit: robot Jaymii, 11 links, 10 joints
Joints:
- joint base_footprint_to_center_camera: origin xyz=-.102 0 1.499 rpy=0 .8 0 -> xyz=-.09 0 1.445 rpy=0 .5 0
- joint base_footprint_to_gps: origin xyz=-.102 .178 1.499 rpy=0 0 0 -> xyz=-0.07112 0.178 1.445 rpy=0 0 0
- joint base_footprint_to_imu: origin xyz=-0.102 0.155 1.499 rpy=0 0 0 -> xyz= 0.279 -0.05 1.445 rpy=0 0 0
- joint base_footprint_to_lidar: origin xyz=.610 -.013 .597 rpy=0 0 0 -> xyz=0.635 0.0 .597 rpy=0 0 0
