Commit message: move covariances over

File: igvc_description/urdf/jessi.urdf (robot description, URDF)
Before this commit: robot Jaymii, 11 links, 10 joints
Joints:
- joint base_footprint_to_imu: origin xyz= 0.279 -0.05 1.445 rpy=0 0 0 -> xyz= 0 0 .2032 rpy=0 0 0

Commit message: update transform for bottom imu

File: igvc_description/urdf/jessi.urdf (robot description, URDF)
Before this commit: robot Jaymii, 11 links, 10 joints
Joints:
- joint base_footprint_to_imu: origin xyz= 0.279 -0.05 1.445 rpy=0 0 0 -> xyz==0.0549656 0 0.2032254 rpy=0 0 0

Commit message: fix typo in urdf

File: igvc_description/urdf/jessi.urdf (robot description, URDF)
Before this commit: robot Jaymii, 11 links, 10 joints
Joints:
- joint base_footprint_to_imu: origin xyz==0.0549656 0 0.2032254 rpy=0 0 0 -> xyz=0.0549656 0 0.2032254 rpy=0 0 0

Commit message: modify urdf to account for new imu transforms. Add frame_id to YostLabs driver

File: igvc_description/urdf/jessi.urdf (robot description, URDF)
Before this commit: robot Jaymii, 11 links, 10 joints
Links:
- added link magnetometer; visual box size=0.1 0.1 0.1
Joints:
- added joint base_footprint_to_magnetometer: type fixed, parent base_footprint, child magnetometer, origin xyz=-0.07112 0 1.23698 rpy=0 0 0, axis 0 0 0
- joint base_footprint_to_imu: origin xyz==0.0549656 0 0.2032254 rpy=0 0 0 -> xyz= 0.054991 0 0.2032254 rpy=0 0 0
