Commit message: added two camera and one imu

File: igvc_description/urdf/jessii.urdf.xacro (robot description, xacro)
@@ -26,9 +26,21 @@
   <xacro:property name="caster_mass" value="1.0"/>
   <xacro:property name="caster_x" value="0.612978"/>
-  <!-- camera params -->
-  <xacro:property name="camera_y" value="0.0"/>
-  <xacro:property name="camera_x" value="0.216371"/>
-  <xacro:property name="camera_pitch" value="0.0"/>
-  <xacro:property name="camera_z" value="1.354330"/>
+  <!-- center camera params -->
+  <xacro:property name="center_camera_y" value="0.0"/>
+  <xacro:property name="center_camera_x" value="0.216371"/>
+  <xacro:property name="center_camera_pitch" value="0.0"/>
+  <xacro:property name="center_camera_z" value="1.354330"/>
+  <!-- right camera params -->
+  <xacro:property name="right_camera_y" value="0.3"/>
+  <xacro:property name="right_camera_x" value="0.216371"/>
+  <xacro:property name="right_camera_pitch" value="0.0"/>
+  <xacro:property name="right_camera_yaw" value="0.0"/>
+  <xacro:property name="right_camera_z" value="1.354330"/>
+  <!-- left camera params -->
+  <xacro:property name="left_camera_y" value="-0.3"/>
+  <xacro:property name="left_camera_x" value="0.216371"/>
+  <xacro:property name="left_camera_pitch" value="0.0"/>
+  <xacro:property name="left_camera_yaw" value="0.0"/>
+  <xacro:property name="left_camera_z" value="1.354330"/>
   <!-- lidar params -->
   <xacro:property name="lidar_pitch" value="0.174533"/>
@@ -41,8 +53,12 @@
   <xacro:property name="gps_y" value="0.198120"/>
   <xacro:property name="gps_x" value="0.216371"/>
-  <!-- imu -->
+  <!-- imu bottom -->
   <xacro:property name="imu_z" value="1.354330"/>
   <xacro:property name="imu_y" value="-0.198120"/>
   <xacro:property name="imu_x" value="0.216371"/>
+  <!-- imu top -->
+  <xacro:property name="magnetometer_z" value="1.354330"/>
+  <xacro:property name="magnetometer_y" value="-0.198120"/>
+  <xacro:property name="magnetometer_x" value="0.216371"/>
   <!-- gives small geometry so it show up in rviz -->
   <xacro:macro name="null_link">
@@ -215,5 +231,5 @@
   </link>
   <joint name="base_link_to_center_cam" type="fixed">
-      <origin xyz="${camera_x} ${camera_y} ${camera_z}" rpy="0 ${camera_pitch} 0" />
+      <origin xyz="${center_camera_x} ${center_camera_y} ${center_camera_z}" rpy="0 ${center_camera_pitch} 0" />
       <parent link="base_link"/>
       <child link="center_cam"/>
@@ -267,4 +283,124 @@
       </sensor>
   </gazebo>
+  <link name="right_cam">
+      <visual>
+          <geometry>
+              <box size="0.1 0.1 0.1"/>
+          </geometry>
+      </visual>
+  </link>
+  <joint name="base_link_to_right_cam" type="fixed">
+      <origin xyz="${right_camera_x} ${right_camera_y} ${right_camera_z}" rpy="0 ${right_camera_pitch} ${right_camera_yaw}" />
+      <parent link="base_link"/>
+      <child link="right_cam"/>
+  </joint>
+  <!-- the optical joint is in the correct frame for transforms -->
+  <link name="right_cam_optical"/>
+  <joint name="right_cam_optical_joint" type="fixed">
+      <parent link="right_cam"/>
+      <child link="right_cam_optical"/>
+      <origin xyz="0 0 0" rpy="-1.5708 0 -1.5708"/>
+  </joint>
+  <gazebo reference="right_cam">
+      <sensor name="right_cam_sensor" type="camera">
+          <camera>
+              <horizontal_fov>1.2290609</horizontal_fov>
+              <image>
+                <width>1920</width>
+                <height>1080</height>
+              </image>
+              <clip>
+                <near>0.1</near>
+                <far>100</far>
+              </clip>
+              <!--
+                  <distortion>
+                  <k1>-0.25</k1>
+                  <k2>0.12</k2>
+                  <k3>0.0</k3>
+                  <p1>-0.00028</p1>
+                  <p2>-0.00005</p2>
+                  <center>0.5 0.5</center>
+                  </distortion>
+              -->
+          </camera>
+          <always_on>1</always_on>
+          <update_rate>30</update_rate>
+          <plugin name="camera_controller" filename="libgazebo_ros_camera.so">
+              <alwaysOn>true</alwaysOn>
+              <updateRate>30</updateRate>
+              <cameraName>right_cam</cameraName>
+              <imageTopicName>image_raw</imageTopicName>
+              <cameraInfoTopicName>camera_info</cameraInfoTopicName>
+              <frameName>right_cam_optical</frameName>
+              <hackBaseline>0.0</hackBaseline>
+              <distortionK1>0.0</distortionK1>
+              <distortionK2>0.0</distortionK2>
+              <distortionK3>0.0</distortionK3>
+              <distortionT1>0.0</distortionT1>
+              <distortionT2>0.0</distortionT2>
+          </plugin>
+      </sensor>
+  </gazebo>
+  <link name="left_cam">
+      <visual>
+          <geometry>
+              <box size="0.1 0.1 0.1"/>
+          </geometry>
+      </visual>
+  </link>
+  <joint name="base_link_to_left_cam" type="fixed">
+      <origin xyz="${left_camera_x} ${left_camera_y} ${left_camera_z}" rpy="0 ${left_camera_pitch} ${left_camera_yaw}" />
+      <parent link="base_link"/>
+      <child link="left_cam"/>
+  </joint>
+  <!-- the optical joint is in the correct frame for transforms -->
+  <link name="left_cam_optical"/>
+  <joint name="left_cam_optical_joint" type="fixed">
+      <parent link="left_cam"/>
+      <child link="left_cam_optical"/>
+      <origin xyz="0 0 0" rpy="-1.5708 0 -1.5708"/>
+  </joint>
+  <gazebo reference="left_cam">
+      <sensor name="left_cam_sensor" type="camera">
+          <camera>
+              <horizontal_fov>1.2290609</horizontal_fov>
+              <image>
+                <width>1920</width>
+                <height>1080</height>
+              </image>
+              <clip>
+                <near>0.1</near>
+                <far>100</far>
+              </clip>
+              <!--
+                  <distortion>
+                  <k1>-0.25</k1>
+                  <k2>0.12</k2>
+                  <k3>0.0</k3>
+                  <p1>-0.00028</p1>
+                  <p2>-0.00005</p2>
+                  <center>0.5 0.5</center>
+                  </distortion>
+              -->
+          </camera>
+          <always_on>1</always_on>
+          <update_rate>30</update_rate>
+          <plugin name="camera_controller" filename="libgazebo_ros_camera.so">
+              <alwaysOn>true</alwaysOn>
+              <updateRate>30</updateRate>
+              <cameraName>left_cam</cameraName>
+              <imageTopicName>image_raw</imageTopicName>
+              <cameraInfoTopicName>camera_info</cameraInfoTopicName>
+              <frameName>left_cam_optical</frameName>
+              <hackBaseline>0.0</hackBaseline>
+              <distortionK1>0.0</distortionK1>
+              <distortionK2>0.0</distortionK2>
+              <distortionK3>0.0</distortionK3>
+              <distortionT1>0.0</distortionT1>
+              <distortionT2>0.0</distortionT2>
+          </plugin>
+      </sensor>
+  </gazebo>
     <!-- base of the robot, should be ground level directly below center points of wheels -->
   <link name="base_link">
@@ -329,4 +465,18 @@
     <axis xyz="0 0 0"/>
   </joint>
+  <link name="magnetometer">
+    <visual>
+      <geometry>
+        <!-- TODO dimensions -->
+        <box size="0.1 0.1 0.1"/>
+      </geometry>
+    </visual>
+  </link>
+  <joint name="base_link_to_magnetometer" type="fixed">
+    <parent link="base_link"/>
+    <child link="magnetometer"/>
+    <origin xyz="${magnetometer_x} ${magnetometer_y} ${magnetometer_z}" rpy="0 0 0"/>
+    <axis xyz="0 0 0"/>
+  </joint>
   <link name="imu">
     <visual>
@@ -366,4 +516,24 @@
       <frameId>imu</frameId>
       <topicName>/imu</topicName>
+      <rpyOffset>0 0 0</rpyOffset>
+      <xyzOffset>0 0 0</xyzOffset>
+      <gaussianNoise>0.00000001</gaussianNoise>
+      <accelDrift>0.00000001 0.00000001 0.00000001</accelDrift>
+      <accelDriftFrequency>0.00000001 0.00000001 0.00000001</accelDriftFrequency>
+      <accelGaussianNoise>0.00000001 0.00000001 0.00000001</accelGaussianNoise>
+      <rateDrift>0.0 0.0 0.0</rateDrift>
+      <rateDriftFrequency>0.0 0.0 0.0</rateDriftFrequency>
+      <rateGaussianNoise>0.0 0.0 0.0</rateGaussianNoise>
+      <headingDrift>0.0 0.0 0.0</headingDrift>
+      <headingDriftFrequency>0.0 0.0 0.0</headingDriftFrequency>
+      <headingGaussianNoise>0.0 0.0 0.0</headingGaussianNoise>
+      <yawOffset>1.5707963</yawOffset>
+    </plugin>
+    <plugin filename="libhector_gazebo_ros_imu.so" name="imu">
+      <serviceName>/magnetometer/calibrate</serviceName>
+      <updateRate>200.0</updateRate>
+      <bodyName>magnetometer</bodyName>
+      <frameId>magnetometer</frameId>
+      <topicName>/magnetometer</topicName>
       <rpyOffset>0 0 0</rpyOffset>
       <xyzOffset>0 0 0</xyzOffset>

Commit message: fixed comments in xacro file and changed relative frames for cameras

File: igvc_description/urdf/jessii.urdf.xacro (robot description, xacro)
@@ -25,11 +25,12 @@
   <xacro:property name="caster_radius" value="0.1016"/>
   <xacro:property name="caster_mass" value="1.0"/>
+  <!-- how far forward from base_link it is -->
   <xacro:property name="caster_x" value="0.612978"/>
-  <!-- center camera params -->
+  <!-- center camera params, relative to the magnetometer -->
   <xacro:property name="center_camera_y" value="0.0"/>
   <xacro:property name="center_camera_x" value="0.216371"/>
   <xacro:property name="center_camera_pitch" value="0.0"/>
   <xacro:property name="center_camera_z" value="1.354330"/>
-  <!-- right camera params -->
+  <!-- right camera params, relative to the magnetometer -->
   <xacro:property name="right_camera_y" value="0.3"/>
   <xacro:property name="right_camera_x" value="0.216371"/>
@@ -37,5 +38,5 @@
   <xacro:property name="right_camera_yaw" value="0.0"/>
   <xacro:property name="right_camera_z" value="1.354330"/>
-  <!-- left camera params -->
+  <!-- left camera params, relative to the magnetometer -->
   <xacro:property name="left_camera_y" value="-0.3"/>
   <xacro:property name="left_camera_x" value="0.216371"/>
@@ -43,5 +44,5 @@
   <xacro:property name="left_camera_yaw" value="0.0"/>
   <xacro:property name="left_camera_z" value="1.354330"/>
-  <!-- lidar params -->
+  <!-- lidar params relative to base_link-->
   <xacro:property name="lidar_pitch" value="0.174533"/>
   <xacro:property name="lidar_x" value="0.680364"/>
@@ -49,13 +50,13 @@
   <xacro:property name="lidar_hz" value="10"/>
   <xacro:property name="lidar_samples" value="500"/>
-  <!-- gps -->
+  <!-- gps, relative to base_link -->
   <xacro:property name="gps_z" value="1.354330"/>
   <xacro:property name="gps_y" value="0.198120"/>
   <xacro:property name="gps_x" value="0.216371"/>
-  <!-- imu bottom -->
+  <!-- imu bottom, relative to base_link -->
   <xacro:property name="imu_z" value="1.354330"/>
   <xacro:property name="imu_y" value="-0.198120"/>
   <xacro:property name="imu_x" value="0.216371"/>
-  <!-- imu top -->
+  <!-- imu top, relative to base_link -->
   <xacro:property name="magnetometer_z" value="1.354330"/>
   <xacro:property name="magnetometer_y" value="-0.198120"/>
@@ -230,7 +231,7 @@
       </visual>
   </link>
-  <joint name="base_link_to_center_cam" type="fixed">
+  <joint name="magnetometer_to_center_cam" type="fixed">
       <origin xyz="${center_camera_x} ${center_camera_y} ${center_camera_z}" rpy="0 ${center_camera_pitch} 0" />
-      <parent link="base_link"/>
+      <parent link="magnetometer"/>
       <child link="center_cam"/>
   </joint>
@@ -245,4 +246,5 @@
       <sensor name="center_cam_sensor" type="camera">
           <camera>
+              <!-- hov in radians -->
               <horizontal_fov>1.2290609</horizontal_fov>
               <image>
@@ -290,7 +292,7 @@
       </visual>
   </link>
-  <joint name="base_link_to_right_cam" type="fixed">
+  <joint name="magnetometer_to_right_cam" type="fixed">
       <origin xyz="${right_camera_x} ${right_camera_y} ${right_camera_z}" rpy="0 ${right_camera_pitch} ${right_camera_yaw}" />
-      <parent link="base_link"/>
+      <parent link="magnetometer"/>
       <child link="right_cam"/>
   </joint>
@@ -305,4 +307,5 @@
       <sensor name="right_cam_sensor" type="camera">
           <camera>
+              <!-- hov in radians -->
               <horizontal_fov>1.2290609</horizontal_fov>
               <image>
@@ -350,7 +353,7 @@
       </visual>
   </link>
-  <joint name="base_link_to_left_cam" type="fixed">
+  <joint name="magnetometer_to_left_cam" type="fixed">
       <origin xyz="${left_camera_x} ${left_camera_y} ${left_camera_z}" rpy="0 ${left_camera_pitch} ${left_camera_yaw}" />
-      <parent link="base_link"/>
+      <parent link="magnetometer"/>
       <child link="left_cam"/>
   </joint>
@@ -365,4 +368,5 @@
       <sensor name="left_cam_sensor" type="camera">
           <camera>
+              <!-- hov in radians -->
               <horizontal_fov>1.2290609</horizontal_fov>
               <image>

Commit message: updated parameters to jessii

File: igvc_description/urdf/jessii.urdf.xacro (robot description, xacro)
@@ -29,19 +29,19 @@
   <!-- center camera params, relative to the magnetometer -->
   <xacro:property name="center_camera_y" value="0.0"/>
-  <xacro:property name="center_camera_x" value="0.216371"/>
+  <xacro:property name="center_camera_x" value="0.0"/>
   <xacro:property name="center_camera_pitch" value="0.0"/>
-  <xacro:property name="center_camera_z" value="1.354330"/>
+  <xacro:property name="center_camera_z" value="0.043942"/>
   <!-- right camera params, relative to the magnetometer -->
-  <xacro:property name="right_camera_y" value="0.3"/>
-  <xacro:property name="right_camera_x" value="0.216371"/>
-  <xacro:property name="right_camera_pitch" value="0.0"/>
-  <xacro:property name="right_camera_yaw" value="0.0"/>
-  <xacro:property name="right_camera_z" value="1.354330"/>
+  <xacro:property name="right_camera_y" value="-0.33147"/>
+  <xacro:property name="right_camera_x" value="0.019812"/>
+  <xacro:property name="right_camera_pitch" value="1.06465"/>
+  <xacro:property name="right_camera_yaw" value="-1.13446"/>
+  <xacro:property name="right_camera_z" value="0"/>
   <!-- left camera params, relative to the magnetometer -->
-  <xacro:property name="left_camera_y" value="-0.3"/>
-  <xacro:property name="left_camera_x" value="0.216371"/>
-  <xacro:property name="left_camera_pitch" value="0.0"/>
-  <xacro:property name="left_camera_yaw" value="0.0"/>
-  <xacro:property name="left_camera_z" value="1.354330"/>
+  <xacro:property name="left_camera_y" value="0.33147"/>
+  <xacro:property name="left_camera_x" value="0.019812"/>
+  <xacro:property name="left_camera_pitch" value="1.06465"/>
+  <xacro:property name="left_camera_yaw" value="1.13446"/>
+  <xacro:property name="left_camera_z" value="0.0"/>
   <!-- lidar params relative to base_link-->
   <xacro:property name="lidar_pitch" value="0.174533"/>
@@ -55,10 +55,10 @@
   <xacro:property name="gps_x" value="0.216371"/>
   <!-- imu bottom, relative to base_link -->
-  <xacro:property name="imu_z" value="1.354330"/>
-  <xacro:property name="imu_y" value="-0.198120"/>
-  <xacro:property name="imu_x" value="0.216371"/>
+  <xacro:property name="imu_z" value="0.221742"/>
+  <xacro:property name="imu_y" value="0.0"/>
+  <xacro:property name="imu_x" value="-0.024638"/>
   <!-- imu top, relative to base_link -->
-  <xacro:property name="magnetometer_z" value="1.354330"/>
-  <xacro:property name="magnetometer_y" value="-0.198120"/>
+  <xacro:property name="magnetometer_z" value="1.238758"/>
+  <xacro:property name="magnetometer_y" value="0.0"/>
   <xacro:property name="magnetometer_x" value="0.216371"/>
   <!-- gives small geometry so it show up in rviz -->

Commit message: Created motor model to model motor dynamics

File: igvc_description/urdf/jessii.urdf.xacro (robot description, xacro)
@@ -16,5 +16,5 @@
   <!-- wheel acuator limits -->
   <xacro:property name="drive_wheel_eff_limit" value="8"/>
-  <xacro:property name="drive_wheel_vel_limit" value="20"/>
+  <xacro:property name="drive_wheel_vel_limit" value="10"/>
   <!-- drive shock params-->
   <!-- how far the drive wheel shock can move (m)-->

Commit message: initial refactor of perception node to integrate sim_detector changes

File: igvc_description/urdf/jessii.urdf.xacro (robot description, xacro)
@@ -30,5 +30,5 @@
   <xacro:property name="center_camera_y" value="0.0"/>
   <xacro:property name="center_camera_x" value="0.0"/>
-  <xacro:property name="center_camera_pitch" value="0.0"/>
+  <xacro:property name="center_camera_pitch" value="0.628319"/>
   <xacro:property name="center_camera_z" value="0.043942"/>
   <!-- right camera params, relative to the magnetometer -->

Commit message: refactor sim_detector to segment images from all 3 cameras

File: igvc_description/urdf/jessii.urdf.xacro (robot description, xacro)
@@ -30,5 +30,5 @@
   <xacro:property name="center_camera_y" value="0.0"/>
   <xacro:property name="center_camera_x" value="0.0"/>
-  <xacro:property name="center_camera_pitch" value="0.628319"/>
+  <xacro:property name="center_camera_pitch" value="0.418879"/>
   <xacro:property name="center_camera_z" value="0.043942"/>
   <!-- right camera params, relative to the magnetometer -->

Commit message: fix base_link->base_footprint in the urdf. provide heading data to navsat_transform_node. Comment out ground_truth_publisher

File: igvc_description/urdf/jessii.urdf.xacro (robot description, xacro)
@@ -420,8 +420,8 @@
     <material>Gazebo/Grey</material>
   </gazebo>
-  <joint name="base_footprint_to_base_link" type="fixed">
-    <parent link="base_footprint"/>
-    <child link="base_link"/>
-    <origin xyz="0.0 0.0 ${drive_tire_diameter / 2}" rpy="0 0 0"/>
+  <joint name="base_link_to_base_footprint" type="fixed">
+    <parent link="base_link"/>
+    <child link="base_footprint"/>
+    <origin xyz="0.0 0.0 -${drive_tire_diameter / 2}" rpy="0 0 0"/>
     <axis xyz="0 0 0"/>
   </joint>

Commit message: correct imu  msg frame_id. Fuse map odometry estimate into navsat_transform_node

File: igvc_description/urdf/jessii.urdf.xacro (robot description, xacro)
@@ -12,5 +12,5 @@
   <xacro:property name="drive_tire_width" value="0.0762"/>
   <!-- TODO set proper mass values -->
-  <xacro:property name="drive_wheel_mass" value="5.0"/>
+  <xacro:property name="drive_wheel_mass" value="3.62874"/>
   <xacro:property name="wheelbase" value="0.714333"/>
   <!-- wheel acuator limits -->
@@ -538,5 +538,5 @@
       <updateRate>200.0</updateRate>
       <bodyName>magnetometer</bodyName>
-      <frameId>magnetometer</frameId>
+      <frameId>imu</frameId>
       <topicName>/magnetometer</topicName>
       <rpyOffset>0 0 0</rpyOffset>

Commit message: Unified all camera frames to have a "cam" prefix Resized output image in the sim_detector node to match the output size of the neural network Added lines back in to the mapper for simulation

File: igvc_description/urdf/jessii.urdf.xacro (robot description, xacro)
@@ -237,8 +237,8 @@
   </joint>
   <!-- the optical joint is in the correct frame for transforms -->
-  <link name="center_cam_optical"/>
-  <joint name="center_cam_optical_joint" type="fixed">
+  <link name="cam/center_optical"/>
+  <joint name="cam/center_optical_joint" type="fixed">
       <parent link="center_cam"/>
-      <child link="center_cam_optical"/>
+      <child link="cam/center_optical"/>
       <origin xyz="0 0 0" rpy="-1.5708 0 -1.5708"/>
   </joint>
@@ -272,8 +272,8 @@
               <alwaysOn>true</alwaysOn>
               <updateRate>30</updateRate>
-              <cameraName>center_cam</cameraName>
+              <cameraName>cam/center</cameraName>
               <imageTopicName>image_raw</imageTopicName>
               <cameraInfoTopicName>camera_info</cameraInfoTopicName>
-              <frameName>center_cam_optical</frameName>
+              <frameName>cam/center_optical</frameName>
               <hackBaseline>0.0</hackBaseline>
               <distortionK1>0.0</distortionK1>
@@ -298,8 +298,8 @@
   </joint>
   <!-- the optical joint is in the correct frame for transforms -->
-  <link name="right_cam_optical"/>
-  <joint name="right_cam_optical_joint" type="fixed">
+  <link name="cam/right_optical"/>
+  <joint name="cam/right_optical_joint" type="fixed">
       <parent link="right_cam"/>
-      <child link="right_cam_optical"/>
+      <child link="cam/right_optical"/>
       <origin xyz="0 0 0" rpy="-1.5708 0 -1.5708"/>
   </joint>
@@ -333,8 +333,8 @@
               <alwaysOn>true</alwaysOn>
               <updateRate>30</updateRate>
-              <cameraName>right_cam</cameraName>
+              <cameraName>cam/right</cameraName>
               <imageTopicName>image_raw</imageTopicName>
               <cameraInfoTopicName>camera_info</cameraInfoTopicName>
-              <frameName>right_cam_optical</frameName>
+              <frameName>cam/right_optical</frameName>
               <hackBaseline>0.0</hackBaseline>
               <distortionK1>0.0</distortionK1>
@@ -359,8 +359,8 @@
   </joint>
   <!-- the optical joint is in the correct frame for transforms -->
-  <link name="left_cam_optical"/>
-  <joint name="left_cam_optical_joint" type="fixed">
+  <link name="cam/left_optical"/>
+  <joint name="cam/left_optical_joint" type="fixed">
       <parent link="left_cam"/>
-      <child link="left_cam_optical"/>
+      <child link="cam/left_optical"/>
       <origin xyz="0 0 0" rpy="-1.5708 0 -1.5708"/>
   </joint>
@@ -394,8 +394,8 @@
               <alwaysOn>true</alwaysOn>
               <updateRate>30</updateRate>
-              <cameraName>left_cam</cameraName>
+              <cameraName>cam/left</cameraName>
               <imageTopicName>image_raw</imageTopicName>
               <cameraInfoTopicName>camera_info</cameraInfoTopicName>
-              <frameName>left_cam_optical</frameName>
+              <frameName>cam/left_optical</frameName>
               <hackBaseline>0.0</hackBaseline>
               <distortionK1>0.0</distortionK1>
