Commit message: Changes camera frame + topics to use namespaces more, clean up segmented image and camera_info topic, adds camera intrinsics matrix scaling and publishing for sim_detector

File: igvc_description/urdf/jessii.urdf.xacro (robot description, xacro)
@@ -224,5 +224,5 @@
     </gazebo>
   </xacro:macro>
-  <link name="center_cam">
+  <link name="cam/center">
       <visual>
           <geometry>
@@ -234,14 +234,14 @@
       <origin xyz="${center_camera_x} ${center_camera_y} ${center_camera_z}" rpy="0 ${center_camera_pitch} 0" />
       <parent link="magnetometer"/>
-      <child link="center_cam"/>
+      <child link="cam/center"/>
   </joint>
   <!-- the optical joint is in the correct frame for transforms -->
   <link name="cam/center_optical"/>
   <joint name="cam/center_optical_joint" type="fixed">
-      <parent link="center_cam"/>
+      <parent link="cam/center"/>
       <child link="cam/center_optical"/>
       <origin xyz="0 0 0" rpy="-1.5708 0 -1.5708"/>
   </joint>
-  <gazebo reference="center_cam">
+  <gazebo reference="cam/center">
       <sensor name="center_cam_sensor" type="camera">
           <camera>
@@ -272,6 +272,6 @@
               <alwaysOn>true</alwaysOn>
               <updateRate>30</updateRate>
-              <cameraName>cam/center</cameraName>
-              <imageTopicName>image_raw</imageTopicName>
+              <cameraName>cam/center/raw</cameraName>
+              <imageTopicName>image</imageTopicName>
               <cameraInfoTopicName>camera_info</cameraInfoTopicName>
               <frameName>cam/center_optical</frameName>
@@ -285,5 +285,5 @@
       </sensor>
   </gazebo>
-  <link name="right_cam">
+  <link name="cam/right">
       <visual>
           <geometry>
@@ -295,14 +295,14 @@
       <origin xyz="${right_camera_x} ${right_camera_y} ${right_camera_z}" rpy="0 ${right_camera_pitch} ${right_camera_yaw}" />
       <parent link="magnetometer"/>
-      <child link="right_cam"/>
+      <child link="cam/right"/>
   </joint>
   <!-- the optical joint is in the correct frame for transforms -->
   <link name="cam/right_optical"/>
   <joint name="cam/right_optical_joint" type="fixed">
-      <parent link="right_cam"/>
+      <parent link="cam/right"/>
       <child link="cam/right_optical"/>
       <origin xyz="0 0 0" rpy="-1.5708 0 -1.5708"/>
   </joint>
-  <gazebo reference="right_cam">
+  <gazebo reference="cam/right">
       <sensor name="right_cam_sensor" type="camera">
           <camera>
@@ -333,6 +333,6 @@
               <alwaysOn>true</alwaysOn>
               <updateRate>30</updateRate>
-              <cameraName>cam/right</cameraName>
-              <imageTopicName>image_raw</imageTopicName>
+              <cameraName>cam/right/raw</cameraName>
+              <imageTopicName>image</imageTopicName>
               <cameraInfoTopicName>camera_info</cameraInfoTopicName>
               <frameName>cam/right_optical</frameName>
@@ -346,5 +346,5 @@
       </sensor>
   </gazebo>
-  <link name="left_cam">
+  <link name="cam/left">
       <visual>
           <geometry>
@@ -356,14 +356,14 @@
       <origin xyz="${left_camera_x} ${left_camera_y} ${left_camera_z}" rpy="0 ${left_camera_pitch} ${left_camera_yaw}" />
       <parent link="magnetometer"/>
-      <child link="left_cam"/>
+      <child link="cam/left"/>
   </joint>
   <!-- the optical joint is in the correct frame for transforms -->
   <link name="cam/left_optical"/>
   <joint name="cam/left_optical_joint" type="fixed">
-      <parent link="left_cam"/>
+      <parent link="cam/left"/>
       <child link="cam/left_optical"/>
       <origin xyz="0 0 0" rpy="-1.5708 0 -1.5708"/>
   </joint>
-  <gazebo reference="left_cam">
+  <gazebo reference="cam/left">
       <sensor name="left_cam_sensor" type="camera">
           <camera>
@@ -394,6 +394,6 @@
               <alwaysOn>true</alwaysOn>
               <updateRate>30</updateRate>
-              <cameraName>cam/left</cameraName>
-              <imageTopicName>image_raw</imageTopicName>
+              <cameraName>cam/left/raw</cameraName>
+              <imageTopicName>image</imageTopicName>
               <cameraInfoTopicName>camera_info</cameraInfoTopicName>
               <frameName>cam/left_optical</frameName>

Commit message: Changed model:// to package:// so that both rviz and gazebo can resolve paths correctly Changed floating joint to fixed joint as tf doesn't work for floating joints Moved robot_state_publisher from igvc_navigation to igvc_description

File: igvc_description/urdf/jessii.urdf.xacro (robot description, xacro)
@@ -136,10 +136,10 @@
       <visual>
         <geometry>
-          <mesh filename="model://urdf/meshes/Wheel.dae"/>
+          <mesh filename="package://igvc_description/urdf/meshes/Wheel.dae"/>
         </geometry>
       </visual>
       <collision>
         <geometry>
-          <mesh filename="model://urdf/meshes/Wheel.dae"/>
+          <mesh filename="package://igvc_description/urdf/meshes/Wheel.dae"/>
         </geometry>
         <max_contacts>10</max_contacts>
@@ -195,5 +195,5 @@
       </collision>
     </link>
-    <joint name="base_link_to_caster" type="floating">
+    <joint name="base_link_to_caster" type="fixed">
       <parent link="base_link"/>
       <child link="caster"/>
@@ -454,10 +454,10 @@
       <visual>
           <geometry>
-              <mesh filename="model://urdf/meshes/jessi_simple.dae"/>
+              <mesh filename="package://igvc_description/urdf/meshes/jessi_simple.dae"/>
           </geometry>
       </visual>
       <collision>
           <geometry>
-              <mesh filename="model://urdf/meshes/jessi_simple.dae"/>
+              <mesh filename="package://igvc_description/urdf/meshes/jessi_simple.dae"/>
           </geometry>
       </collision>

Commit message: changed values for wheel seperation

File: igvc_description/urdf/jessii.urdf.xacro (robot description, xacro)
@@ -13,5 +13,5 @@
   <!-- TODO set proper mass values -->
   <xacro:property name="drive_wheel_mass" value="5.0"/>
-  <xacro:property name="wheelbase" value="0.714333"/>
+  <xacro:property name="wheelbase" value="0.556"/>
   <!-- wheel acuator limits -->
   <xacro:property name="drive_wheel_eff_limit" value="8"/>

Commit message: Add a working swervi submodule

File: igvc_description/urdf/jessii.urdf.xacro (robot description, xacro)
@@ -84,5 +84,5 @@
       <axis xyz="0 0 -1"/>
       <limit lower="${-drive_wheel_travel / 2}" upper="${drive_wheel_travel / 2}"
-             effort="${drive_shock_eff_limit}" velocity="${drive_shock_vel_limit}"/>
+              effort="${drive_shock_eff_limit}" velocity="${drive_shock_vel_limit}"/>
       <!-- TODO tune for actual shocks -->
       <!-- damping = viscous dampening coeff -->
@@ -407,5 +407,5 @@
       </sensor>
   </gazebo>
-    <!-- base of the robot, should be ground level directly below center points of wheels -->
+  <!-- base of the robot, should be ground level directly below center points of wheels -->
   <link name="base_link">
     <xacro:null_link/>

File: igvc_description/urdf/swervi.urdf.xacro (robot description, xacro)
@@ -1,61 +1,46 @@
 <?xml version="1.0"?>
-<robot name="igvc_platform" xmlns:xacro="http://www.ros.org/wiki/xacro">
-    <xacro:property name="wheel_mass" value="1" />
-    <xacro:property name="wheel_width" value="1" />
-    <xacro:property name="tire_diameter" value="1" />
-    <material name="blue">
-        <color rgba="0 0 0.8 1"/>
-    </material>
-    <material name="black">
-        <color rgba="0 0 0 1"/>
-    </material>
-    <material name="white">
-        <color rgba="1 1 1 1"/>
-    </material>
+<robot name="Swervi" xmlns:xacro="http://www.ros.org/wiki/xacro">
+    <xacro:include filename="swerve_module.urdf.xacro"/>
+    <xacro:property name="wheel_diameter" value="0.275" />
+    <!-- base of the robot, should be ground level, centered on the robot -->
     <link name="base_link">
-        <visual>
-            <geometry>
-                <cylinder length="0.6" radius="0.2"/>
-            </geometry>
-            <material name="blue"/>
-        </visual>
-        <collision>
-            <geometry>
-                <cylinder length="0.6" radius="0.2"/>
-            </geometry>
-        </collision>
-        <inertial>
-            <mass value="10"/>
-            <inertia ixx="0.4" ixy="0.0" ixz="0.0" iyy="0.4" iyz="0.0" izz="0.2"/>
-        </inertial>
+        <xacro:null_link/>
     </link>
-    <link name="wheel">
-        <visual>
-            <geometry>
-                <mesh filename="package://igvc_description/urdf/meshes/Wheel.dae"/>
-            </geometry>
-            <origin rpy= "1.57075 0 0" xyz = "0 0 0"/>
-        </visual>
-        <collision>
-            <geometry>
-                <mesh filename="package://igvc_description/urdf/meshes/Wheel.dae"/>
-            </geometry>
-            <origin rpy= "1.57075 0 0" xyz = "0 0 0"/>
-        </collision>
-        <inertial>
-            <mass value="1"/>
-            <inertia  ixx="1"
-                      ixy="0.0"
-                      ixz="0.0"
-                      iyy="1"
-                      iyz="0.0"
-                      izz="1" />
-        </inertial>
+    <gazebo reference="base_link">
+        <material>Gazebo/Grey</material>
+    </gazebo>
+    <link name="base_footprint">
+        <xacro:null_link/>
     </link>
-    <joint name="base_to_wheel" type="continuous">
-        <parent link="base_link"/>
-        <child link="wheel"/>
-        <origin xyz="0 -0.25 -0.3"/>
-        <axis xyz="0 1 0"/>
+    <gazebo reference="base_footprint">
+        <material>Gazebo/Grey</material>
+    </gazebo>
+    <joint name="base_footprint_to_base_link" type="fixed">
+        <parent link="base_footprint"/>
+        <child link="base_link"/>
+        <origin xyz="0.0 0.0 ${wheel_diameter / 2}" rpy="0 0 0"/>
     </joint>
+    <xacro:swerve_module prefix="tl" x_pos="0" y_pos="0"/> -->
+    <!-- Just Used for testing -->
+    <link name="world"/>
+    <joint name="world_to_base_footprint" type="fixed">
+        <parent link="world"/>
+        <child link="base_footprint"/>
+    </joint>
+    <gazebo>
+        <plugin name="gazebo_ros_control" filename="libgazebo_ros_control.so">
+            <robotSimType>gazebo_ros_control/DefaultRobotHWSim</robotSimType>
+        </plugin>
+        <plugin name="p3d_base_controller" filename="libgazebo_ros_p3d.so">
+            <alwaysOn>true</alwaysOn>
+            <updateRate>200.0</updateRate>
+            <bodyName>base_footprint</bodyName>
+            <topicName>ground_truth/state_raw</topicName>
+            <gaussianNoise>0.00</gaussianNoise>
+            <frameName>world</frameName>
+            <!-- origin is at spawn location -->
+            <xyzOffset>0 0 0</xyzOffset>
+            <rpyOffset>0 0 0</rpyOffset>
+        </plugin>
+    </gazebo>
 </robot>
