Commit message: Add chassis, four swerve submodules, and lidar to swervi

File: igvc_description/urdf/swerve_module.urdf.xacro (robot description, xacro)
@@ -1,34 +1,4 @@
 <?xml version="1.0"?>
 <robot name="Swervi" xmlns:xacro="http://www.ros.org/wiki/xacro">
-    <!-- constants -->
-    <xacro:property name="M_PI" value="3.1415926535897931" />
-    <!-- geometry params -->
-    <xacro:property name="wheel_mass" value="15" />
-    <xacro:property name="wheel_width" value="0.0762" />
-    <xacro:property name="wheel_diameter" value="0.305"/>
-    <xacro:property name="swivel_radius" value="0.1375" />
-    <xacro:property name="swivel_length" value="0.17272" />
-    <xacro:property name="swivel_mass" value="1" />
-    <xacro:property name="wheel_swivel_offset" value="0.02" />
-    <!-- wheel acuator limits -->
-    <xacro:property name="drive_wheel_eff_limit" value="8"/>
-    <xacro:property name="drive_wheel_vel_limit" value="10"/>
-    <!-- drive shock params-->
-    <!-- how far the drive wheel shock can move (m)-->
-    <xacro:property name="drive_wheel_travel" value="0.1"/>
-    <xacro:property name="drive_shock_eff_limit" value="500.0"/>
-    <xacro:property name="drive_shock_vel_limit" value="0.1"/>
-    <!-- gives small geometry so it show up in rviz -->
-    <xacro:macro name="null_link">
-        <inertial>
-            <mass value="0.001"/>
-            <inertia ixx="0.001" ixy="0" ixz="0" iyy="0.001" iyz="0" izz="0.001"/>
-        </inertial>
-        <visual>
-            <geometry>
-                <box size="0.01 0.01 0.01"/>
-            </geometry>
-        </visual>
-    </xacro:macro>
     <!-- makes shock for drive wheel -->
     <xacro:macro name="drive_shock" params="prefix x_pos y_pos">
@@ -36,11 +6,11 @@
             <parent link="base_link"/>
             <child link="${prefix}_swerve_base"/>
-            <origin xyz="${x_pos} ${y_pos} 0 "
+            <origin xyz="${x_pos} ${y_pos} ${wheel_radius+swivel_height}"
                     rpy="0 0 0"/>
             <axis xyz="0 0 -1"/>
             <limit lower="${-drive_wheel_travel / 2}" upper="${drive_wheel_travel / 2}"
                     effort="${drive_shock_eff_limit}" velocity="${drive_shock_vel_limit}"/>
-            <dynamics damping="100" friction="1.0"
-                        spring_stiffness="113832.44275" spring_reference="0.08"/>
+            <dynamics damping="${drive_shock_damping}" friction="${drive_shock_friction}"
+                        spring_stiffness="${drive_spring_stiffness}" spring_reference="${drive_shock_spring_ref}"/>
         </joint>
         <transmission name="${prefix}_drive_shock_trans">
@@ -65,5 +35,5 @@
             <parent link="${prefix}_swerve_base"/>
             <child link="${prefix}_swivel_axle"/>
-            <origin xyz="0 0 ${-swivel_length/2}" rpy="0 0 0"/>
+            <origin xyz="0 0 ${-swivel_height/2}" rpy="0 0 0"/>
         </joint>
         <link name="${prefix}_swivel_axle">
@@ -74,16 +44,16 @@
             <child link="${prefix}_swerve_swivel"/>
             <axis xyz="0 0 -1"/>
-            <limit effort="${drive_wheel_eff_limit}" velocity="${drive_wheel_vel_limit}"/>
-            <dynamics damping="0.001" friction="0.5"/>
+            <limit effort="${max_torque_swivel}" velocity="${max_vel_swivel}"/>
+            <dynamics damping="${swivel_damping}" friction="${swivel_friction}"/>
         </joint>
         <link name="${prefix}_swerve_swivel">
             <visual>
                 <geometry>
-                    <cylinder length="${swivel_length}" radius="${swivel_radius}"/>
+                    <cylinder length="${swivel_height}" radius="${swivel_radius}"/>
                 </geometry>
             </visual>
             <inertial>
                 <mass value="${swivel_mass}"/>
-                <inertia ixx="0.4" ixy="0.0" ixz="0.0" iyy="0.4" iyz="0.0" izz="0.2"/>
+                <inertia ixx="${swivel_Ixx}" ixy="0.0" ixz="0.0" iyy="${swivel_Iyy}" iyz="0.0" izz="${swivel_Izz}"/>
             </inertial>
         </link>
@@ -99,7 +69,7 @@
         </transmission>
         <joint name="${prefix}_wheel_offset" type="fixed">
-            <parent link="${prefix}_swivel_axle"/>
+            <parent link="${prefix}_swerve_swivel"/>
             <child link="${prefix}_wheel_axle"/>
-            <origin xyz="0 0 ${-swivel_length/2}" rpy="0 0 0"/>
+            <origin xyz="0 0 ${-swivel_height/2}" rpy="0 0 0"/>
         </joint>
         <link name="${prefix}_wheel_axle">
@@ -112,7 +82,7 @@
             <child link="${prefix}_wheel"/>
             <origin xyz="0 0 0" rpy="${M_PI / 2} 0 0"/>
-            <axis xyz="0 0 0"/>
-            <limit effort="${drive_wheel_eff_limit}" velocity="${drive_wheel_vel_limit}"/>
-            <dynamics damping="0.001" friction="0.5"/>
+            <axis xyz="0 0 1"/>
+            <limit effort="${max_torque_hub}" velocity="${max_vel_hub}"/>
+            <dynamics damping="${wheel_damping}" friction="${wheel_friction}"/>
         </joint>
         <transmission name="${prefix}_axle_trans">
@@ -131,10 +101,10 @@
             <visual>
                 <geometry>
-                    <mesh filename="package://igvc_description/urdf/meshes/Wheel.dae"/>
+                    <mesh filename="package://igvc_description/urdf/meshes/swervi_tire.dae"/>
                 </geometry>
             </visual>
             <collision>
                 <geometry>
-                    <mesh filename="package://igvc_description/urdf/meshes/Wheel.dae"/>
+                    <mesh filename="package://igvc_description/urdf/meshes/swervi_tire.dae"/>
                 </geometry>
                 <max_contacts>10</max_contacts>
@@ -153,12 +123,11 @@
             </collision>
             <inertial>
-                <origin xyz="0 0 0" />
                 <mass value="${wheel_mass}"/>
-                <inertia  ixx="${1 / 12 * wheel_mass * wheel_width**2 + 1/4 * wheel_mass * (wheel_diameter / 2)**2}"
+                <inertia  ixx="${wheel_Ixx_Iyy}"
                         ixy="0.0"
                         ixz="0.0"
-                        iyy="${1 / 12 * wheel_mass * wheel_width**2 + 1/4 * wheel_mass * (wheel_diameter / 2)**2}"
+                        iyy="${wheel_Ixx_Iyy}"
                         iyz="0.0"
-                        izz="${1/2 * wheel_mass * (wheel_diameter / 2)**2}" />
+                        izz="${wheel_Izz}" />
             </inertial>
         </link>

File: igvc_description/urdf/swervi.urdf.xacro (robot description, xacro)
@@ -1,6 +1,7 @@
 <?xml version="1.0"?>
 <robot name="Swervi" xmlns:xacro="http://www.ros.org/wiki/xacro">
+    <xacro:include filename="swervi_prop.urdf.xacro"/>
     <xacro:include filename="swerve_module.urdf.xacro"/>
-    <xacro:property name="wheel_diameter" value="0.275" />
+    <xacro:include filename="$(find velodyne_description)/urdf/VLP-16.urdf.xacro"/>
     <!-- base of the robot, should be ground level, centered on the robot -->
     <link name="base_link">
@@ -19,13 +20,63 @@
         <parent link="base_footprint"/>
         <child link="base_link"/>
-        <origin xyz="0.0 0.0 ${wheel_diameter / 2}" rpy="0 0 0"/>
+        <origin xyz="0.0 0.0 0.0" rpy="0 0 0"/>
     </joint>
-    <xacro:swerve_module prefix="tl" x_pos="0" y_pos="0"/> -->
-    <!-- Just Used for testing -->
+    <link name="chassis">
+        <inertial>
+            <mass value="${chassis_mass}" />
+            <origin xyz="0 0 0" rpy="0 0 0"/>
+            <!-- approximate the intertial matrix as a sphere -->
+            <inertia  ixx="${chassis_Ixx}" ixy="0.0" ixz="0.0"
+                        iyy="${chassis_Iyy}" iyz="0.0"
+                        izz="${chassis_Izz}" />
+        </inertial>
+        <visual>
+            <geometry>
+                <mesh filename="package://igvc_description/urdf/meshes/swervi_chassis.dae"/>
+            </geometry>
+        </visual>
+        <collision>
+            <geometry>
+                <mesh filename="package://igvc_description/urdf/meshes/swervi_chassis.dae"/>
+            </geometry>
+        </collision>
+    </link>
+    <joint name="base_link_to_chassis" type="fixed">
+        <parent link="base_link"/>
+        <child link="chassis"/>
+        <origin xyz="0.0 0.0 ${chassis_offset_z}" rpy="${M_PI / 2} 0 ${M_PI / 2}"/>
+    </joint>
+    <gazebo reference="chassis">
+        <material>Gazebo/Grey</material>
+        <mu1>0.2</mu1>
+        <mu2>0.2</mu2>
+    </gazebo>
+    <xacro:swerve_module prefix="fl" x_pos="${wheel_offset_x}" y_pos="${-wheel_offset_y}"/>
+    <xacro:swerve_module prefix="bl" x_pos="${-wheel_offset_x}" y_pos="${-wheel_offset_y}"/>
+    <xacro:swerve_module prefix="br" x_pos="${-wheel_offset_x}" y_pos="${wheel_offset_y}"/>
+    <xacro:swerve_module prefix="fr" x_pos="${wheel_offset_x}" y_pos="${wheel_offset_y}"/>
+    <link name="lidar_support">
+        <visual>
+            <geometry>
+                <box size="${lidar_support_x_dim} ${lidar_support_y_dim} ${lidar_support_z_dim}"/>
+            </geometry>
+        </visual>
+    </link>
+    <joint name="base_link_to_lidar_support" type="fixed">
+        <parent link="base_link"/>
+        <child link="lidar_support"/>
+        <origin xyz="${lidar_x/2} 0.0 ${lidar_z-lidar_support_z_dim/2}" rpy="0.0 0.0 0.0"/>
+    </joint>
+    <!-- collision range = min sensing distance -->
+    <!-- gpu does gpu acceleration -->
+    <xacro:VLP-16 parent="base_link" name="lidar" topic="/velodyne_points" hz="${lidar_hz}" samples="${lidar_samples}" gpu="$(arg gpu)">
+        <origin xyz="${lidar_x} 0.0 ${lidar_z}" rpy="0 ${lidar_pitch} 0" />
+    </xacro:VLP-16>
+    <!-- Just Used for testing
     <link name="world"/>
     <joint name="world_to_base_footprint" type="fixed">
         <parent link="world"/>
         <child link="base_footprint"/>
-    </joint>
+    </joint> -->
     <gazebo>
         <plugin name="gazebo_ros_control" filename="libgazebo_ros_control.so">

Commit message: Fixed directions for swerve drive and swervi

File: igvc_description/urdf/swerve_module.urdf.xacro (robot description, xacro)
@@ -43,5 +43,5 @@
             <parent link="${prefix}_swivel_axle"/>
             <child link="${prefix}_swerve_swivel"/>
-            <axis xyz="0 0 -1"/>
+            <axis xyz="0 0 1"/>
             <limit effort="${max_torque_swivel}" velocity="${max_vel_swivel}"/>
             <dynamics damping="${swivel_damping}" friction="${swivel_friction}"/>
@@ -82,5 +82,5 @@
             <child link="${prefix}_wheel"/>
             <origin xyz="0 0 0" rpy="${M_PI / 2} 0 0"/>
-            <axis xyz="0 0 1"/>
+            <axis xyz="0 0 -1"/>
             <limit effort="${max_torque_hub}" velocity="${max_vel_hub}"/>
             <dynamics damping="${wheel_damping}" friction="${wheel_friction}"/>

File: igvc_description/urdf/swervi.urdf.xacro (robot description, xacro)
@@ -52,8 +52,8 @@
         <mu2>0.2</mu2>
     </gazebo>
-    <xacro:swerve_module prefix="fl" x_pos="${wheel_offset_x}" y_pos="${-wheel_offset_y}"/>
-    <xacro:swerve_module prefix="bl" x_pos="${-wheel_offset_x}" y_pos="${-wheel_offset_y}"/>
-    <xacro:swerve_module prefix="br" x_pos="${-wheel_offset_x}" y_pos="${wheel_offset_y}"/>
-    <xacro:swerve_module prefix="fr" x_pos="${wheel_offset_x}" y_pos="${wheel_offset_y}"/>
+    <xacro:swerve_module prefix="fl" x_pos="${wheel_offset_x}" y_pos="${wheel_offset_y}"/>
+    <xacro:swerve_module prefix="bl" x_pos="${-wheel_offset_x}" y_pos="${wheel_offset_y}"/>
+    <xacro:swerve_module prefix="br" x_pos="${-wheel_offset_x}" y_pos="${-wheel_offset_y}"/>
+    <xacro:swerve_module prefix="fr" x_pos="${wheel_offset_x}" y_pos="${-wheel_offset_y}"/>
     <link name="lidar_support">
         <visual>
